File: power_supply_2.kicad_sch (KiCad schematic)
At the start: 36 parts, among them U1 LM317, U2 LM337

Commit message: cosmetics
Other:
- note added: "Chassis Ground"
- note added: "Regulated Power Supply"
- moved on the sheet: C1, C10, C11, C12, C13, C14, C2, C3, C4, C5, C6, C7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
